File: hw/pc_mainboard/ethernet.kicad_sch (KiCad schematic)
At the start: 0 parts

Commit message: Added PHY research
Parts:
- added U3: phy_MXL86110I-AQB-R, QFN40_5X5_MXL, symbol pc_mainboard:phy_MXL86110I-AQB-R
Other:
- title: (none) -> Phy
Changed lines of the file:
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@@
 	(generator_version "8.0")
 	(paper "A4")
+	(title_block
+		(title "Phy")
+	)
+	(symbol
+		(lib_id "pc_mainboard:phy_MXL86110I-AQB-R")
+		(at 109.22 68.58 0)
+		(unit 1)
+		(exclude_from_sim no)
+		(in_bom yes)
+		(on_board yes)
+		(dnp no)
+		(fields_autoplaced yes)
+		(property "Reference" "U3"
+			(at 147.32 58.42 0)
+			(effects
+				(font
+					(size 1.524 1.524)
+				)
+			)
+		)
+		(property "Value" "phy_MXL86110I-AQB-R"
+			(at 147.32 60.96 0)
+			(effects
+				(font
+					(size 1.524 1.524)
+				)
+			)
+		)
+		(property "Footprint" "QFN40_5X5_MXL"
+			(at 109.22 68.58 0)
+			(effects
+				(font
+					(size 1.27 1.27)
+					(italic yes)
+				)
+				(hide yes)
+			)
+		)
+		(property "Datasheet" "MXL86110I-AQB-R"
+			(at 109.22 68.58 0)
+			(effects
+				(font
+					(size 1.27 1.27)
+					(italic yes)
+				)
+				(hide yes)
+			)
+		)
+		(property "Description" ""
+			(at 109.22 68.58 0)
+			(effects
+				(font
+					(size 1.27 1.27)
+				)
+				(hide yes)
+			)
+		)
+		(pin "6"
+		)
+		(pin "39"
+		)
+		(pin "3"
+		)
+		(pin "14"
+		)
+		(pin "27"
+		)
+		(pin "29"
+		)
+		(pin "7"
+		)
+		(pin "5"
+		)
+		(pin "16"
+		)
+		(pin "20"
+		)
+		(pin "37"
+		)
+		(pin "40"
+		)
+		(pin "12"
+		)
+		(pin "21"
+		)
+		(pin "41"
+		)
+		(pin "24"
+		)
+		(pin "26"
+		)
+		(pin "9"
+		)
+		(pin "1"
+		)
+		(pin "28"
+		)
+		(pin "10"
+		)
+		(pin "25"
+		)
+		(pin "2"
+		)
+		(pin "19"
+		)
+		(pin "35"
+		)
+		(pin "38"
+		)
+		(pin "23"
+		)
+		(pin "34"
+		)
+		(pin "11"
+		)
+		(pin "13"
+		)
+		(pin "30"
+		)
+		(pin "31"
+		)
+		(pin "36"
+		)
+		(pin "22"
+		)
+		(pin "4"
+		)
+		(pin "8"
+		)
+		(pin "33"
+		)
+		(pin "32"
+		)
+		(pin "17"
+		)
+		(pin "15"
+		)
+		(pin "18"
+		)
+		(instances
+			(project ""
+				(path "/69a74940-cd00-4a75-bd5b-2bda9e86219a/36ea05e7-a91a-429d-8bc8-710554747042"
+					(reference "U3")
+					(unit 1)
+				)
+			)
+		)
+	)
 )
