File: hw/pc_mainboard/ram.kicad_sch (KiCad schematic)
At the start: 0 parts

Commit message: Added RAM information
Parts:
- added U2: MT41K256M16TW-107:P, FBGA96_8X14_MRN, symbol pc_mainboard:MT41K256M16TW-107_P
Other:
- title: (none) -> RAM

Commit message: RAM Schematic Capture (#39)
Parts:
- added C12, C13, C14, C16, C17, C18, C19, C20, C21, C22, C23, C24, C25, C26, C27, C28, C29, C30, C31: 100n, symbol Device:C
- added C15: 10u, symbol Device:C
- added R10: 100, symbol Device:R
- added R11, R12, R8: 10k, symbol Device:R
- added R9: 240, symbol Device:R
Connections:
- net GND: now reaches U2.97 (EPAD)
- net GND: now also U2.A9 (VSS), U2.B1 (VSSQ), U2.B3 (VSS), U2.B9 (VSSQ), U2.D1 (VSSQ), U2.D8 (VSSQ), U2.E1 (VSS), U2.E2 (VSSQ), U2.E8 (VSSQ), U2.F9 (VSSQ), U2.G1 (VSSQ), U2.G8 (VSS), U2.G9 (VSSQ), U2.J2 (VSS), U2.J8 (VSS), U2.M1 (VSS), U2.M9 (VSS), U2.P1 (VSS), U2.P9 (VSS), U2.T1 (VSS), U2.T9 (VSS), C12.2, C13.2, C14.2, C15.2, C16.2, C17.2, C18.2, C19.2, C20.2, C21.2, C22.2, C23.2, C24.2, C25.2, C26.2, C27.2, C28.2, C29.2, C30.2, C31.2, R11.2, R8.2, R9.2
- net +1V35: now reaches U2.A1 (VDDQ)
- net +1V35: now also U2.A8 (VDDQ), U2.B2 (VDD), U2.C1 (VDDQ), U2.C9 (VDDQ), U2.D2 (VDDQ), U2.D9 (VDD), U2.E9 (VDDQ), U2.F1 (VDDQ), U2.G7 (VDD), U2.H2 (VDDQ), U2.H9 (VDDQ), U2.K2 (VDD), U2.K8 (VDD), U2.N1 (VDD), U2.N9 (VDD), U2.R1 (VDD), U2.R9 (VDD), C14.1, C15.1, C16.1, C17.1, C18.1, C19.1, C20.1, C21.1, C22.1, C23.1, C24.1, C25.1, C26.1, C27.1, C28.1, C29.1, C30.1, C31.1
- net DDR_D.13: now reaches U2.A2 (DQ13)
- net DDR_D.15: now reaches U2.A3 (DQ15)
- net DDR_D.12: now reaches U2.A7 (DQ12)
- net DDR_CTRL.UDQS-: now reaches U2.B7 (*UDQS)
- net DDR_D.14: now reaches U2.B8 (DQ14)
- net DDR_D.11: now reaches U2.C2 (DQ11)
- net DDR_D.9: now reaches U2.C3 (DQ9)
- net DDR_CTRL.UDQS+: now reaches U2.C7 (UDQS)
- net DDR_D.10: now reaches U2.C8 (DQ10)
- net DDR_CTRL.UDM: now reaches U2.D3 (UDM)
- net DDR_D.8: now reaches U2.D7 (DQ8)
- net DDR_D.0: now reaches U2.E3 (DQ0)
- net DDR_CTRL.LDM: now reaches U2.E7 (LDM)
- net DDR_D.2: now reaches U2.F2 (DQ2)
- net DDR_CTRL.LDQS+: now reaches U2.F3 (LDQS)
- net DDR_D.1: now reaches U2.F7 (DQ1)
- net DDR_D.3: now reaches U2.F8 (DQ3)
- net DDR_D.6: now reaches U2.G2 (DQ6)
- net DDR_CTRL.LDQS-: now reaches U2.G3 (*LDQS)
- net V_REF_DDR: now reaches U2.H1 (VREFDQ)
- net V_REF_DDR: now also U2.M8 (VREFCA), C12.1, C13.1, R12.1
- net DDR_D.4: now reaches U2.H3 (DQ4)
- net DDR_D.7: now reaches U2.H7 (DQ7)
- net DDR_D.5: now reaches U2.H8 (DQ5)
- net ~{DDR_CTRL.RAS}: now reaches U2.J3 (*RAS)
- net DDR_CTRL.CK+: now reaches U2.J7 (CK)
- net DDR_CTRL.CK+: now also R10.1
- net DDR_CTRL.ODT: now reaches U2.K1 (ODT)
- net ~{DDR_CTRL.CAS}: now reaches U2.K3 (*CAS)
- net DDR_CTRL.CK-: now reaches U2.K7 (*CK)
- net DDR_CTRL.CK-: now also R10.2
- net DDR_CKE: now reaches U2.K9 (CKE)
- net DDR_CKE: now also R11.1, R12.2
- net ~{DDR_CTRL.CS}: now reaches U2.L2 (*CS)
- net ~{DDR_CTRL.WE}: now reaches U2.L3 (*WE)
- net DDR_A.10: now reaches U2.L7 (A10/AP)
- net DDR_ZQ: now reaches U2.L8 (ZQ)
- net DDR_ZQ: now also R9.1
- net DDR_BA.0: now reaches U2.M2 (BA0)
- net DDR_BA.2: now reaches U2.M3 (BA2)
- net DDR_A.3: now reaches U2.N2 (A3)
- net DDR_A.0: now reaches U2.N3 (A0)
- net DDR_A.12: now reaches U2.N7 (A12/*BC)
- net DDR_BA.1: now reaches U2.N8 (BA1)
- net DDR_A.5: now reaches U2.P2 (A5)
- net DDR_A.2: now reaches U2.P3 (A2)
- net DDR_A.1: now reaches U2.P7 (A1)
- net DDR_A.4: now reaches U2.P8 (A4)
- net DDR_A.7: now reaches U2.R2 (A7)
- net DDR_A.9: now reaches U2.R3 (A9)
- net DDR_A.11: now reaches U2.R7 (A11)
- net DDR_A.6: now reaches U2.R8 (A6)
- net ~{DDR_RESET}: now reaches U2.T2 (*RESET)
- net ~{DDR_RESET}: now also R8.1
- net DDR_A.13: now reaches U2.T3 (A13)
- net DDR_A.14: now reaches U2.T7 (A14)
- net DDR_A.8: now reaches U2.T8 (A8)
Other:
- note added: "DDR Address Bus"
- note added: "DDR Bank Address Bus"
- note added: "DDR Config"
- note added: "DDR Control Bus"
- note added: "DDR Data Bus"
- note added: "RAM Power Consort"
- note added: "VREF Power Consort"
- moved on the sheet: U2
