File: hw/pc_mainboard/eeprom.kicad_sch (KiCad schematic)
At the start: 2 parts

Commit message: v1 HDMI Transmitter Schematic
Other:
- note removed: "Reference: shorthand for numerical value types 0b -- binary (0000, etc) 0x -- hexidecimal (FF, etc)"
Changed lines of the file:
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@@
 	(text "I2C address format for this component kind: 0b1010xxx+RW\nThis component address: 0b1010000"
 		(exclude_from_sim no)
-		(at 115.57 129.032 0)
+		(at 116.332 125.476 0)
 		(effects
 			(font
-				(size 1.27 1.27)
-			)
-			(justify left top)
-		)
-	)
-	(text "Reference: shorthand for numerical value types\n0b -- binary (0000, etc)\n0x -- hexidecimal (FF, etc)"
-		(exclude_from_sim no)
-		(at 116.078 137.668 0)
-		(effects
-			(font
