File: hw/pc_mainboard/eeprom.kicad_sch (KiCad schematic)
At the start: 2 parts

Commit message: Schematic capture Flash
Other:
- note added: "I2C Address: 0b1010000X"
- note removed: "I2C address format for this component kind: 0b1010xxx+RW This component address: 0b1010000"
- note removed: "Reference: shorthand for numerical value types 0b -- binary (0000, etc) 0x -- hexidecimal (FF, etc)"
- moved on the sheet: C32, CR1
