File: hw/pc_mainboard/pc_mainboard.kicad_sch (KiCad schematic)
At the start: 0 parts

Commit message: v1 HDMI Transmitter Schematic
Other:
- added sheet HDMI Transmitter (hdmi_transmitter.kicad_sch)
Changed lines of the file:
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@@
+	)
+	(sheet
+		(at 374.65 224.79)
+		(size 31.75 24.13)
+		(exclude_from_sim no)
+		(in_bom yes)
+		(on_board yes)
+		(dnp no)
+		(fields_autoplaced yes)
+		(stroke
+			(width 0.1524)
+			(type solid)
+		)
+		(fill
+			(color 0 0 0 0.0000)
+		)
+		(property "Sheetname" "HDMI Transmitter"
+			(at 374.65 224.0784 0)
+			(effects
+				(font
+					(size 1.27 1.27)
+				)
+				(justify left bottom)
+			)
+		)
+		(property "Sheetfile" "hdmi_transmitter.kicad_sch"
+			(at 374.65 249.5046 0)
+			(effects
+				(font
+					(size 1.27 1.27)
+				)
+				(justify left top)
+			)
+		)
+		(instances
+			(project "pc_mainboard"
+				(path "/69a74940-cd00-4a75-bd5b-2bda9e86219a"
+					(page "14")
+				)
+			)
+		)
 	)
 	(sheet
