File: hw/pc_mainboard/pc_mainboard.kicad_sch (KiCad schematic)
At the start: 0 parts

Commit message: Schematic capture Flash
Other:
- sheet flash ports: added FLASH[0..3], FLASH_SCLK, ~{FLASH_CS}; removed none
Changed lines of the file:
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@@
 	)
 	(sheet
-		(at 306.07 170.18)
-		(size 50.8 40.64)
+		(at 306.07 184.15)
+		(size 16.51 12.7)
 		(exclude_from_sim no)
 		(in_bom yes)
@@
 		)
 		(property "Sheetname" "flash"
-			(at 306.07 169.4684 0)
+			(at 306.07 183.4384 0)
 			(effects
 				(font
@@
 		)
 		(property "Sheetfile" "flash.kicad_sch"
-			(at 306.07 211.4046 0)
+			(at 306.07 197.4346 0)
 			(effects
 				(font
@@
 			)
 		)
+		(pin "FLASH[0..3]" bidirectional
+			(at 306.07 187.96 180)
+			(effects
+				(font
+					(size 1.27 1.27)
+				)
+				(justify left)
+			)
+		)
+		(pin "FLASH_SCLK" input
+			(at 306.07 190.5 180)
+			(effects
+				(font
+					(size 1.27 1.27)
+				)
+				(justify left)
+			)
+		)
+		(pin "~{FLASH_CS}" input
+			(at 306.07 193.04 180)
+			(effects
+				(font
+					(size 1.27 1.27)
+				)
+				(justify left)
+			)
+		)
