File: hw/pc_mainboard/sd_card_interface.kicad_sch (KiCad schematic)
At the start: 0 parts

Commit message: SD card research, updated some formatting (#49)
Parts:
- added J2: sd_card_MEM2067-02-180-00-A_REVB, MEM2067-02-180-00-A_REVB:GCT_MEM2067-02-180-00-A_REVB, symbol pc_mainboard:sd_card_MEM2067-02-180-00-A_REVB
Other:
- title: (none) -> SD Card Interface
Changed lines of the file:
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@@
 	(generator_version "9.0")
 	(paper "A4")
+	(title_block
+		(title "SD Card Interface")
+	)
+	(symbol
+		(lib_id "pc_mainboard:sd_card_MEM2067-02-180-00-A_REVB")
+		(at 134.62 86.36 0)
+		(unit 1)
+		(exclude_from_sim no)
+		(in_bom yes)
+		(on_board yes)
+		(dnp no)
+		(fields_autoplaced yes)
+		(property "Reference" "J2"
+			(at 151.13 89.5349 0)
+			(effects
+				(font
+					(size 1.27 1.27)
+				)
+				(justify left)
+			)
+		)
+		(property "Value" "sd_card_MEM2067-02-180-00-A_REVB"
+			(at 151.13 92.0749 0)
+			(effects
+				(font
+					(size 1.27 1.27)
+				)
+				(justify left)
+			)
+		)
+		(property "Footprint" "MEM2067-02-180-00-A_REVB:GCT_MEM2067-02-180-00-A_REVB"
+			(at 134.62 86.36 0)
+			(effects
+				(font
+					(size 1.27 1.27)
+				)
+				(justify bottom)
+				(hide yes)
+			)
+		)
+		(property "Datasheet" ""
+			(at 134.62 86.36 0)
+			(effects
+				(font
+					(size 1.27 1.27)
+				)
+				(hide yes)
+			)
+		)
+		(property "Description" ""
+			(at 134.62 86.36 0)
+			(effects
+				(font
+					(size 1.27 1.27)
+				)
+				(hide yes)
+			)
+		)
+		(property "MANUFACTURER" "GCT"
+			(at 134.62 86.36 0)
+			(effects
+				(font
+					(size 1.27 1.27)
+				)
+				(justify bottom)
+				(hide yes)
+			)
+		)
+		(pin "2"
+		)
+		(pin "3"
+		)
+		(pin "8"
+		)
+		(pin "7"
+		)
+		(pin "5"
+		)
+		(pin "6"
+		)
+		(pin "11"
+		)
+		(pin "9"
+		)
+		(pin "12"
+		)
+		(pin "4"
+		)
+		(pin "1"
+		)
+		(pin "10"
+		)
+		(instances
+			(project ""
+				(path "/69a74940-cd00-4a75-bd5b-2bda9e86219a/370cf3cd-f652-4cb5-a2e0-db1b03f43015"
+					(reference "J2")
+					(unit 1)
+				)
+			)
+		)
+	)
 )

Commit message: v1 HDMI Transmitter Schematic
Parts:
- renumbered J2 to J3
Other:
- title: SD Card Interface -> HDMI Transmitter
Changed lines of the file:
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@@
 	(paper "A4")
 	(title_block
-		(title "SD Card Interface")
+		(title "HDMI Transmitter")
 	)
 	(symbol
@@
 		(dnp no)
 		(fields_autoplaced yes)
-		(property "Reference" "J2"
+		(property "Reference" "J3"
 			(at 151.13 89.5349 0)
 			(effects
@@
 		(pin "10"
 		)
-		(instances
-			(project ""
-				(path "/69a74940-cd00-4a75-bd5b-2bda9e86219a/370cf3cd-f652-4cb5-a2e0-db1b03f43015"
-					(reference "J2")
-					(unit 1)
-				)
-			)
-		)
 	)
