File: hw/pc_mainboard/flash.kicad_sch (KiCad schematic)
At the start: 0 parts

Commit message: Flash research
Parts:
- added U8: flash_1gb_MX66U1G45GXDI00, CSP24_6X8X1p2_MAC, symbol pc_mainboard:flash_1gb_MX66U1G45GXDI00
Other:
- title: (none) -> Flash
Changed lines of the file:
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@@
 	(generator_version "9.0")
 	(paper "A4")
+	(title_block
+		(title "Flash")
+	)
+	(symbol
+		(lib_id "pc_mainboard:flash_1gb_MX66U1G45GXDI00")
+		(at 124.46 85.09 0)
+		(unit 1)
+		(exclude_from_sim no)
+		(in_bom yes)
+		(on_board yes)
+		(dnp no)
+		(fields_autoplaced yes)
+		(property "Reference" "U8"
+			(at 149.86 74.93 0)
+			(effects
+				(font
+					(size 1.524 1.524)
+				)
+			)
+		)
+		(property "Value" "flash_1gb_MX66U1G45GXDI00"
+			(at 149.86 77.47 0)
+			(effects
+				(font
+					(size 1.524 1.524)
+				)
+			)
+		)
+		(property "Footprint" "CSP24_6X8X1p2_MAC"
+			(at 124.46 85.09 0)
+			(effects
+				(font
+					(size 1.27 1.27)
+					(italic yes)
+				)
+				(hide yes)
+			)
+		)
+		(property "Datasheet" "MX66U1G45GXDI00"
+			(at 124.46 85.09 0)
+			(effects
+				(font
+					(size 1.27 1.27)
+					(italic yes)
+				)
+				(hide yes)
+			)
+		)
+		(property "Description" ""
+			(at 124.46 85.09 0)
+			(effects
+				(font
+					(size 1.27 1.27)
+				)
+				(hide yes)
+			)
+		)
+		(pin "B2"
+		)
+		(pin "D4"
+		)
+		(pin "C2"
+		)
+		(pin "B5"
+		)
+		(pin "C1"
+		)
+		(pin "C3"
+		)
+		(pin "E5"
+		)
+		(pin "E4"
+		)
+		(pin "E2"
+		)
+		(pin "D5"
+		)
+		(pin "C4"
+		)
+		(pin "E1"
+		)
+		(pin "A2"
+		)
+		(pin "D2"
+		)
+		(pin "E3"
+		)
+		(pin "B3"
+		)
+		(pin "A4"
+		)
+		(pin "D1"
+		)
+		(pin "C5"
+		)
+		(pin "B1"
+		)
+		(pin "B4"
+		)
+		(pin "A3"
+		)
+		(pin "A5"
+		)
+		(pin "D3"
+		)
+		(instances
+			(project ""
+				(path "/69a74940-cd00-4a75-bd5b-2bda9e86219a/5acaef94-cd0b-452b-9621-73208b013ff5"
+					(reference "U8")
+					(unit 1)
+				)
+			)
+		)
+	)
 )

Commit message: Schematic capture Flash
Parts:
- added C33: 100n, symbol Device:C
- added R13: 0, symbol Device:R
Connections:
- net at U8.A4 (RESET#): now also R13.2
- net FLASH_SCLK: now reaches U8.B2 (SCLK)
- net GND: now reaches U8.B3 (GND)
- net GND: now also C33.2
- net +1V8: now reaches U8.B4 (VCC)
- net +1V8: now also C33.1, R13.1
- net ~{FLASH_CS}: now reaches U8.C2 (CS#)
- net FLASH.2: now reaches U8.C4 (WP#/SIO2)
- net FLASH.1: now reaches U8.D2 (SO/SIO1)
- net FLASH.0: now reaches U8.D3 (SI/SIO0)
- net FLASH.3: now reaches U8.D4 (NC/SIO3)
